File: _autosave-Science-PSU-PCB.kicad_pcb (KiCad board)
At the start: 2 copper layers, 100 x 90.8 mm, 43 parts, among them J1 XT60-M, J2 ESTOP, J3 ON, J4 XT60-M, J5 XT60-M, J6 XT60-M, J7 Conn_01x04, J8 Screw_Terminal_01x02, J9 Screw_Terminal_01x02, Q1 MMBT3904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

Commit message: PCB Layout and routing.
Routing:
- net /HE_CTRL: track 2.85 -> 30.5 mm
- net /HE_IS: track 36.7 -> 43.7 mm
- net /PWR_CTRL_IS: track 90.9 -> 89.8 mm
Changed lines of the file:
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@@
+	)
+	(segment
+		(start 65.574 87.649)
+		(end 65.525 87.6)
+		(width 0.35)
+		(layer "F.Cu")
+		(net 6)
 	)
 	(segment
@@
 		(net 6)
 	)
+	(segment
+		(start 65.574 94.551)
+		(end 65.574 87.649)
+		(width 0.35)
+		(layer "F.Cu")
+		(net 6)
+	)
 	(via
 		(at 58.8 82.4)
@@
 	)
 	(segment
-		(start 101.1625 73.4)
-		(end 101.1625 107.4375)
-		(width 0.35)
-		(layer "F.Cu")
-		(net 10)
-	)
-	(segment
-		(start 101.1625 107.4375)
-		(end 101 107.6)
+		(start 101.1625 86.6)
+		(end 101.1625 73.4)
 		(width 0.35)
 		(layer "F.Cu")
@@
 	)
 	(via
-		(at 101 107.6)
-		(size 0.6)
-		(drill 0.3)
-		(layers "F.Cu" "B.Cu")
+		(at 101.1625 86.6)
+		(size 0.6)
+		(drill 0.3)
+		(layers "F.Cu" "B.Cu")
+		(net 10)
+	)
+	(segment
+		(start 101.1625 92)
+		(end 99.3625 93.8)
+		(width 0.35)
+		(layer "B.Cu")
+		(net 10)
+	)
+	(segment
+		(start 101.1625 86.6)
+		(end 101.1625 92)
+		(width 0.35)
+		(layer "B.Cu")
+		(net 10)
+	)
+	(segment
+		(start 50.525 102.525)
+		(end 50.525 92.4)
+		(width 0.35)
+		(layer "B.Cu")
+		(net 10)
+	)
+	(segment
+		(start 99.3625 93.8)
+		(end 59.25 93.8)
+		(width 0.35)
+		(layer "B.Cu")
 		(net 10)
 	)
 	(segment
 		(start 99.403415 108)
-		(end 100.6 108)
-		(width 0.35)
-		(layer "B.Cu")
-		(net 10)
-	)
-	(segment
-		(start 50.6 108)
-		(end 98.121585 108)
-		(width 0.35)
-		(layer "B.Cu")
-		(net 10)
-	)
-	(segment
-		(start 99.374915 108.0285)
-		(end 99.403415 108)
-		(width 0.35)
-		(layer "B.Cu")
-		(net 10)
-	)
-	(segment
-		(start 98.150085 108.0285)
 		(end 99.374915 108.0285)
 		(width 0.35)
@@
 	)
 	(segment
-		(start 98.121585 108)
-		(end 98.150085 108.0285)
-		(width 0.35)
-		(layer "B.Cu")
-		(net 10)
-	)
-	(segment
-		(start 100.6 108)
-		(end 101 107.6)
-		(width 0.35)
-		(layer "B.Cu")
-		(net 10)
+		(start 59.25 93.8)
+		(end 50.525 102.525)
+		(width 0.35)
+		(layer "B.Cu")
+		(net 10)
+	)
+	(segment
+		(start 46.925 89.9)
+		(end 62.1 89.9)
+		(width 0.5)
+		(layer "F.Cu")
+		(net 11)
 	)
 	(segment
@@
 		(layer "F.Cu")
 		(net 11)
+	)
+	(segment
+		(start 62.1 89.9)
+		(end 66.2 85.8)
+		(width 0.5)
+		(layer "F.Cu")
+		(net 11)
+	)
+	(segment
+		(start 66.2 85.8)
+		(end 66.2 79.1725)
+		(width 0.5)
+		(layer "F.Cu")
+		(net 11)
